Commit message: --

File: legged_gym/resources/robots/kbot/kbot.urdf (robot description, URDF)
Before this commit: robot kbotv2p0_nohands, 32 links, 31 joints
Links:
- link Torso_Side_Right: geometry collision mesh filename=meshes/Torso_Side_Right.stl; visual mesh filename=meshes/Torso_Side_Right.stl
Joints:
- joint auxiliary_l_foot_joint1: origin xyz=-0.04 0.1 0 rpy=0 0 0 -> xyz=-0.2 -0.005 0 rpy=0 0 0
- joint auxiliary_l_foot_joint2: origin xyz=-0.04 -0.1 0 rpy=0 0 0 -> xyz=0.15 -0.005 0 rpy=0 0 0
- joint auxiliary_l_foot_joint3: origin xyz=0.07 0 0 rpy=0 0 0 -> xyz=0 -0.005 0.10 rpy=0 0 0
- joint auxiliary_l_foot_joint4: origin xyz=-0.15 0 0 rpy=0 0 0 -> xyz=0 -0.005 -0.10 rpy=0 0 0
- joint auxiliary_r_foot_joint1: origin xyz=-0.04 0.1 0 rpy=0 0 0 -> xyz=-0.2 -0.005 0 rpy=0 0 0
- joint auxiliary_r_foot_joint2: origin xyz=-0.04 -0.1 0 rpy=0 0 0 -> xyz=0.15 -0.005 0 rpy=0 0 0
- joint auxiliary_r_foot_joint3: origin xyz=0.07 0 0 rpy=0 0 0 -> xyz=0 -0.005 0.10 rpy=0 0 0
- joint auxiliary_r_foot_joint4: origin xyz=-0.15 0 0 rpy=0 0 0 -> xyz=0 -0.005 -0.10 rpy=0 0 0
- joint keyframe_head_joint: child keyframe_head_link -> Torso_Side_Right; origin xyz=0 0 0.08 rpy=0 0 0 -> xyz=-0.10 -0.10 -0.39 rpy=0 0 0

Commit message: --add kbot

File: legged_gym/resources/robots/kbot/kbot.urdf (robot description, URDF)
Before this commit: robot kbotv2p0_nohands, 32 links, 31 joints
Links:
- removed link KB_C_501X_Left_Bayonet_Adapter_Hard_Stop
- removed link KB_C_501X_Right_Bayonet_Adapter_Hard_Stop
- removed link KB_D_501L_L_LEG_FOOT
- removed link KB_D_501R_R_LEG_FOOT
- removed link KC_C_104L_PitchHardstopDriven
- removed link KC_C_104R_PitchHardstopDriven
- removed link KC_C_202L
- removed link KC_C_202R
- removed link KC_C_401L_L_UpForearmDrive
- removed link KC_C_401R_R_UpForearmDrive
- removed link KC_D_102L_L_Hip_Yoke_Drive
- removed link KC_D_102R_R_Hip_Yoke_Drive
- removed link KC_D_301L_L_Femur_Lower_Drive
- removed link KC_D_301R_R_Femur_Lower_Drive
- removed link KC_D_401L_L_Shin_Drive
- removed link KC_D_401R_R_Shin_Drive
- removed link RS03_3
- removed link RS03_4
- removed link RS03_5
- removed link RS03_6
- removed link Torso_Side_Right
- removed link auxiliary_l_foot_link1
- removed link auxiliary_l_foot_link2
- removed link auxiliary_l_foot_link3
- removed link auxiliary_l_foot_link4
- removed link auxiliary_r_foot_link1
- removed link auxiliary_r_foot_link2
- removed link auxiliary_r_foot_link3
- removed link auxiliary_r_foot_link4
- removed link base
- removed link imu
- added link auxiliary_left_ankle_roll_link1; visual sphere radius=0.01
- added link auxiliary_left_ankle_roll_link2; visual sphere radius=0.01
- added link auxiliary_left_ankle_roll_link3; visual sphere radius=0.01
- added link auxiliary_left_ankle_roll_link4; visual sphere radius=0.01
- added link auxiliary_right_ankle_roll_link1; visual sphere radius=0.01
- added link auxiliary_right_ankle_roll_link2; visual sphere radius=0.01
- added link auxiliary_right_ankle_roll_link3; visual sphere radius=0.01
- added link auxiliary_right_ankle_roll_link4; visual sphere radius=0.01
- added link d435_link
- added link head_link, mass 1.036; collision mesh filename=meshes/head_link.STL; visual mesh filename=meshes/head_link.STL
- added link imu_in_pelvis
- added link imu_in_torso
- added link keyframe_left_ankle_link
- added link keyframe_left_collar_link
- added link keyframe_left_elbow_link
- added link keyframe_left_hip_link
- added link keyframe_left_knee_link
- added link keyframe_left_shoulder_link
- added link keyframe_left_wrist_link
- added link keyframe_pelvis_link
- added link keyframe_right_ankle_link
- added link keyframe_right_collar_link
- added link keyframe_right_elbow_link
- added link keyframe_right_hip_link
- added link keyframe_right_knee_link
- added link keyframe_right_shoulder_link
- added link keyframe_right_wrist_link
- added link keyframe_torso_link
- added link left_ankle_pitch_link, mass 0.074; collision mesh filename=meshes/left_ankle_pitch_link.STL; visual mesh filename=meshes/left_ankle_pitch_link.STL
- added link left_ankle_roll_link, mass 0.608; collision sphere radius=0.005; collision sphere radius=0.005
- added link left_elbow_link, mass 0.6; collision mesh filename=meshes/left_elbow_link.STL; visual mesh filename=meshes/left_elbow_link.STL
- added link left_foot_front_link
- added link left_foot_hind_link
- added link left_foot_mid_link
- added link left_hip_pitch_link, mass 1.35; collision mesh filename=meshes/left_hip_pitch_link.STL; visual mesh filename=meshes/left_hip_pitch_link.STL
- added link left_hip_roll_link, mass 1.52; collision mesh filename=meshes/left_hip_roll_link.STL; visual mesh filename=meshes/left_hip_roll_link.STL
- added link left_hip_yaw_link, mass 1.702; collision mesh filename=meshes/left_hip_yaw_link.STL; visual mesh filename=meshes/left_hip_yaw_link.STL
- added link left_knee_link, mass 1.932; collision mesh filename=meshes/left_knee_link.STL; visual mesh filename=meshes/left_knee_link.STL
- added link left_shoulder_pitch_link, mass 0.718; collision cylinder length=0.05 radius=0.03; visual mesh filename=meshes/left_shoulder_pitch_link.STL
- added link left_shoulder_roll_link, mass 0.643; collision cylinder length=0.03 radius=0.03; visual mesh filename=meshes/left_shoulder_roll_link.STL
- added link left_shoulder_yaw_link, mass 0.734; collision mesh filename=meshes/left_shoulder_yaw_link.STL; visual mesh filename=meshes/left_shoulder_yaw_link.STL
- added link left_wrist_roll_rubber_hand, mass 0.35692864; collision mesh filename=meshes/left_wrist_roll_rubber_hand.STL; visual mesh filename=meshes/left_wrist_roll_rubber_hand.STL
- added link logo_link, mass 0.001; collision mesh filename=meshes/logo_link.STL; visual mesh filename=meshes/logo_link.STL
- added link mid360_link
- added link pelvis, mass 3.813; visual mesh filename=meshes/pelvis.STL
- added link pelvis_contour_link, mass 0.001; collision mesh filename=meshes/pelvis_contour_link.STL; visual mesh filename=meshes/pelvis_contour_link.STL
- added link right_ankle_pitch_link, mass 0.074; collision mesh filename=meshes/right_ankle_pitch_link.STL; visual mesh filename=meshes/right_ankle_pitch_link.STL
- added link right_ankle_roll_link, mass 0.608; collision sphere radius=0.005; collision sphere radius=0.005
- added link right_elbow_link, mass 0.6; collision mesh filename=meshes/right_elbow_link.STL; visual mesh filename=meshes/right_elbow_link.STL
- added link right_foot_front_link
- added link right_foot_hind_link
- added link right_foot_mid_link
- added link right_hip_pitch_link, mass 1.35; collision mesh filename=meshes/right_hip_pitch_link.STL; visual mesh filename=meshes/right_hip_pitch_link.STL
- added link right_hip_roll_link, mass 1.52; collision mesh filename=meshes/right_hip_roll_link.STL; visual mesh filename=meshes/right_hip_roll_link.STL
- added link right_hip_yaw_link, mass 1.702; collision mesh filename=meshes/right_hip_yaw_link.STL; visual mesh filename=meshes/right_hip_yaw_link.STL
- added link right_knee_link, mass 1.932; collision mesh filename=meshes/right_knee_link.STL; visual mesh filename=meshes/right_knee_link.STL
- added link right_shoulder_pitch_link, mass 0.718; collision cylinder length=0.05 radius=0.03; visual mesh filename=meshes/right_shoulder_pitch_link.STL
- added link right_shoulder_roll_link, mass 0.643; collision cylinder length=0.03 radius=0.03; visual mesh filename=meshes/right_shoulder_roll_link.STL
- added link right_shoulder_yaw_link, mass 0.734; collision mesh filename=meshes/right_shoulder_yaw_link.STL; visual mesh filename=meshes/right_shoulder_yaw_link.STL
- added link right_wrist_roll_rubber_hand, mass 0.35692864; collision mesh filename=meshes/right_wrist_roll_rubber_hand.STL; visual mesh filename=meshes/right_wrist_roll_rubber_hand.STL
- added link torso_link, mass 8.562; collision mesh filename=meshes/torso_link.STL; visual mesh filename=meshes/torso_link.STL
- added link waist_support_link, mass 0.001; collision mesh filename=meshes/waist_support_link.STL; visual mesh filename=meshes/waist_support_link.STL
- added link waist_yaw_fixed_link, mass 0.244; visual mesh filename=meshes/waist_yaw_link.STL
- link keyframe_head_link: geometry 
Joints:
- removed joint auxiliary_l_foot_joint1
- removed joint auxiliary_l_foot_joint2
- removed joint auxiliary_l_foot_joint3
- removed joint auxiliary_l_foot_joint4
- removed joint auxiliary_r_foot_joint1
- removed joint auxiliary_r_foot_joint2
- removed joint auxiliary_r_foot_joint3
- removed joint auxiliary_r_foot_joint4
- removed joint base_joint
- removed joint dof_left_ankle_02
- removed joint dof_left_elbow_02
- removed joint dof_left_hip_pitch_04
- removed joint dof_left_hip_roll_03
- removed joint dof_left_hip_yaw_03
- removed joint dof_left_knee_04
- removed joint dof_left_shoulder_pitch_03
- removed joint dof_left_shoulder_roll_03
- removed joint dof_left_shoulder_yaw_02
- removed joint dof_left_wrist_00
- removed joint dof_right_ankle_02
- removed joint dof_right_elbow_02
- removed joint dof_right_hip_pitch_04
- removed joint dof_right_hip_roll_03
- removed joint dof_right_hip_yaw_03
- removed joint dof_right_knee_04
- removed joint dof_right_shoulder_pitch_03
- removed joint dof_right_shoulder_roll_03
- removed joint dof_right_shoulder_yaw_02
- removed joint dof_right_wrist_00
- removed joint frame_imu_site
- added joint auxiliary_left_ankle_roll_joint1: type fixed, parent left_ankle_roll_link, child auxiliary_left_ankle_roll_link1, origin xyz=0.035 0.1 0 rpy=0 0 0
- added joint auxiliary_left_ankle_roll_joint2: type fixed, parent left_ankle_roll_link, child auxiliary_left_ankle_roll_link2, origin xyz=0.035 -0.1 0 rpy=0 0 0
- added joint auxiliary_left_ankle_roll_joint3: type fixed, parent left_ankle_roll_link, child auxiliary_left_ankle_roll_link3, origin xyz=0.2 0 0 rpy=0 0 0
- added joint auxiliary_left_ankle_roll_joint4: type fixed, parent left_ankle_roll_link, child auxiliary_left_ankle_roll_link4, origin xyz=-0.15 0 0 rpy=0 0 0
- added joint auxiliary_right_ankle_roll_joint1: type fixed, parent right_ankle_roll_link, child auxiliary_right_ankle_roll_link1, origin xyz=0.035 0.1 0 rpy=0 0 0
- added joint auxiliary_right_ankle_roll_joint2: type fixed, parent right_ankle_roll_link, child auxiliary_right_ankle_roll_link2, origin xyz=0.035 -0.1 0 rpy=0 0 0
- added joint auxiliary_right_ankle_roll_joint3: type fixed, parent right_ankle_roll_link, child auxiliary_right_ankle_roll_link3, origin xyz=0.2 0 0 rpy=0 0 0
- added joint auxiliary_right_ankle_roll_joint4: type fixed, parent right_ankle_roll_link, child auxiliary_right_ankle_roll_link4, origin xyz=-0.15 0 0 rpy=0 0 0
- added joint d435_joint: type fixed, parent torso_link, child d435_link, origin xyz=0.0576235 0.01753 0.41987 rpy=0 0.8307767239493009 0
- added joint head_joint: type fixed, parent torso_link, child head_link, origin xyz=0.0039635 0 -0.054 rpy=0 0 0
- added joint imu_in_pelvis_joint: type fixed, parent pelvis, child imu_in_pelvis, origin xyz=0.04525 0 -0.08339 rpy=0 0 0
- added joint imu_in_torso_joint: type fixed, parent torso_link, child imu_in_torso, origin xyz=-0.03959 -0.00224 0.13792 rpy=0 0 0
- added joint keyframe_left_ankle_joint: type fixed, parent left_ankle_roll_link, child keyframe_left_ankle_link, origin xyz=0 0 0 rpy=0 0 0
- added joint keyframe_left_collar_joint: type fixed, parent left_shoulder_pitch_link, child keyframe_left_collar_link, origin xyz=0 0 0.02 rpy=0 0 0
- added joint keyframe_left_elbow_joint: type fixed, parent left_elbow_link, child keyframe_left_elbow_link, origin xyz=0 0 0 rpy=0 0 0
- added joint keyframe_left_hip_joint: type fixed, parent left_hip_roll_link, child keyframe_left_hip_link, origin xyz=0 0 0 rpy=0 0 0
- added joint keyframe_left_knee_joint: type fixed, parent left_knee_link, child keyframe_left_knee_link, origin xyz=0 0 0 rpy=0 0 0
- added joint keyframe_left_shoulder_joint: type fixed, parent left_shoulder_roll_link, child keyframe_left_shoulder_link, origin xyz=0 0 0 rpy=0 0 0
- added joint keyframe_left_wrist_joint: type fixed, parent left_wrist_roll_rubber_hand, child keyframe_left_wrist_link, origin xyz=0 0 0 rpy=0 0 0
- added joint keyframe_pelvis_joint: type fixed, parent pelvis, child keyframe_pelvis_link, origin xyz=0 0 -0.075 rpy=0 0 0
- added joint keyframe_right_ankle_joint: type fixed, parent right_ankle_roll_link, child keyframe_right_ankle_link, origin xyz=0 0 0 rpy=0 0 0
- added joint keyframe_right_collar_joint: type fixed, parent right_shoulder_pitch_link, child keyframe_right_collar_link, origin xyz=0 0 0.02 rpy=0 0 0
- added joint keyframe_right_elbow_joint: type fixed, parent right_elbow_link, child keyframe_right_elbow_link, origin xyz=0 0 0 rpy=0 0 0
- added joint keyframe_right_hip_joint: type fixed, parent right_hip_roll_link, child keyframe_right_hip_link, origin xyz=0 0 0 rpy=0 0 0
- added joint keyframe_right_knee_joint: type fixed, parent right_knee_link, child keyframe_right_knee_link, origin xyz=0 0 0 rpy=0 0 0
- added joint keyframe_right_shoulder_joint: type fixed, parent right_shoulder_roll_link, child keyframe_right_shoulder_link, origin xyz=0 0 0 rpy=0 0 0
- added joint keyframe_right_wrist_joint: type fixed, parent right_wrist_roll_rubber_hand, child keyframe_right_wrist_link, origin xyz=0 0 0 rpy=0 0 0
- added joint keyframe_torso_joint: type fixed, parent torso_link, child keyframe_torso_link, origin xyz=0 0 0.2 rpy=0 0 0
- added joint left_ankle_pitch_joint: type revolute, parent left_knee_link, child left_ankle_pitch_link, origin xyz=0 -9.4445E-05 -0.30001 rpy=0 0 0, axis 0 1 0, limit lower=-0.87267 upper=0.5236 effort=50 velocity=37
- added joint left_ankle_roll_joint: type revolute, parent left_ankle_pitch_link, child left_ankle_roll_link, origin xyz=0 0 -0.017558 rpy=0 0 0, axis 1 0 0, limit lower=-0.2618 upper=0.2618 effort=50 velocity=37
- added joint left_elbow_joint: type revolute, parent left_shoulder_yaw_link, child left_elbow_link, origin xyz=0.015783 0 -0.080518 rpy=0 0 0, axis 0 1 0, limit lower=-1.0472 upper=2.0944 effort=25 velocity=37
- added joint left_foot_front_joint: type fixed, parent left_ankle_pitch_link, child left_foot_front_link, origin xyz=0.18 0 -0.06 rpy=0 0 0
- added joint left_foot_hind_joint: type fixed, parent left_ankle_pitch_link, child left_foot_hind_link, origin xyz=-0.09 0 -0.06 rpy=0 0 0
- added joint left_foot_mid_joint: type fixed, parent left_ankle_pitch_link, child left_foot_mid_link, origin xyz=0.0 0 -0.06 rpy=0 0 0
- added joint left_hip_pitch_joint: type revolute, parent pelvis, child left_hip_pitch_link, origin xyz=0 0.064452 -0.1027 rpy=0 0 0, axis 0 1 0, limit lower=-2.5307 upper=2.8798 effort=88 velocity=32
- added joint left_hip_roll_joint: type revolute, parent left_hip_pitch_link, child left_hip_roll_link, origin xyz=0 0.052 -0.030465 rpy=0 -0.1749 0, axis 1 0 0, limit lower=-0.5236 upper=2.9671 effort=88 velocity=32
- added joint left_hip_yaw_joint: type revolute, parent left_hip_roll_link, child left_hip_yaw_link, origin xyz=0.025001 0 -0.12412 rpy=0 0 0, axis 0 0 1, limit lower=-2.7576 upper=2.7576 effort=88 velocity=32
- added joint left_knee_joint: type revolute, parent left_hip_yaw_link, child left_knee_link, origin xyz=-0.078273 0.0021489 -0.17734 rpy=0 0.1749 0, axis 0 1 0, limit lower=-0.087267 upper=2.8798 effort=139 velocity=20
- added joint left_shoulder_pitch_joint: type revolute, parent torso_link, child left_shoulder_pitch_link, origin xyz=0.0039563 0.10022 0.23778 rpy=0.27931 5.4949E-05 -0.00019159, axis 0 1 0, limit lower=-3.0892 upper=2.6704 effort=25 velocity=37
- added joint left_shoulder_roll_joint: type revolute, parent left_shoulder_pitch_link, child left_shoulder_roll_link, origin xyz=0 0.038 -0.013831 rpy=-0.27925 0 0, axis 1 0 0, limit lower=-1.5882 upper=2.2515 effort=25 velocity=37
- added joint left_shoulder_yaw_joint: type revolute, parent left_shoulder_roll_link, child left_shoulder_yaw_link, origin xyz=0 0.00624 -0.1032 rpy=0 0 0, axis 0 0 1, limit lower=-2.618 upper=2.618 effort=25 velocity=37
- added joint left_wrist_roll_joint: type revolute, parent left_elbow_link, child left_wrist_roll_rubber_hand, origin xyz=0.100 0.00188791 -0.010 rpy=0 0 0, axis 1 0 0, limit lower=-1.972222054 upper=1.972222054 effort=25 velocity=37
- added joint logo_joint: type fixed, parent torso_link, child logo_link, origin xyz=0.0039635 0 -0.054 rpy=0 0 0
- added joint mid360_joint: type fixed, parent torso_link, child mid360_link, origin xyz=0.0002835 0.00003 0.40618 rpy=0 0.04014257279586953 0
- added joint pelvis_contour_joint: type fixed, parent pelvis, child pelvis_contour_link
- added joint right_ankle_pitch_joint: type revolute, parent right_knee_link, child right_ankle_pitch_link, origin xyz=0 9.4445E-05 -0.30001 rpy=0 0 0, axis 0 1 0, limit lower=-0.87267 upper=0.5236 effort=50 velocity=37
- added joint right_ankle_roll_joint: type revolute, parent right_ankle_pitch_link, child right_ankle_roll_link, origin xyz=0 0 -0.017558 rpy=0 0 0, axis 1 0 0, limit lower=-0.2618 upper=0.2618 effort=50 velocity=37
- added joint right_elbow_joint: type revolute, parent right_shoulder_yaw_link, child right_elbow_link, origin xyz=0.015783 0 -0.080518 rpy=0 0 0, axis 0 1 0, limit lower=-1.0472 upper=2.0944 effort=25 velocity=37
- added joint right_foot_front_joint: type fixed, parent right_ankle_pitch_link, child right_foot_front_link, origin xyz=0.18 0 -0.06 rpy=0 0 0
- added joint right_foot_hind_joint: type fixed, parent right_ankle_pitch_link, child right_foot_hind_link, origin xyz=-0.09 0 -0.06 rpy=0 0 0
- added joint right_foot_mid_joint: type fixed, parent right_ankle_pitch_link, child right_foot_mid_link, origin xyz=0.0 0 -0.06 rpy=0 0 0
- added joint right_hip_pitch_joint: type revolute, parent pelvis, child right_hip_pitch_link, origin xyz=0 -0.064452 -0.1027 rpy=0 0 0, axis 0 1 0, limit lower=-2.5307 upper=2.8798 effort=88 velocity=32
- added joint right_hip_roll_joint: type revolute, parent right_hip_pitch_link, child right_hip_roll_link, origin xyz=0 -0.052 -0.030465 rpy=0 -0.1749 0, axis 1 0 0, limit lower=-2.9671 upper=0.5236 effort=88 velocity=32
- added joint right_hip_yaw_joint: type revolute, parent right_hip_roll_link, child right_hip_yaw_link, origin xyz=0.025001 0 -0.12412 rpy=0 0 0, axis 0 0 1, limit lower=-2.7576 upper=2.7576 effort=88 velocity=32
- added joint right_knee_joint: type revolute, parent right_hip_yaw_link, child right_knee_link, origin xyz=-0.078273 -0.0021489 -0.17734 rpy=0 0.1749 0, axis 0 1 0, limit lower=-0.087267 upper=2.8798 effort=139 velocity=20
- added joint right_shoulder_pitch_joint: type revolute, parent torso_link, child right_shoulder_pitch_link, origin xyz=0.0039563 -0.10021 0.23778 rpy=-0.27931 5.4949E-05 0.00019159, axis 0 1 0, limit lower=-3.0892 upper=2.6704 effort=25 velocity=37
- added joint right_shoulder_roll_joint: type revolute, parent right_shoulder_pitch_link, child right_shoulder_roll_link, origin xyz=0 -0.038 -0.013831 rpy=0.27925 0 0, axis 1 0 0, limit lower=-2.2515 upper=1.5882 effort=25 velocity=37
- added joint right_shoulder_yaw_joint: type revolute, parent right_shoulder_roll_link, child right_shoulder_yaw_link, origin xyz=0 -0.00624 -0.1032 rpy=0 0 0, axis 0 0 1, limit lower=-2.618 upper=2.618 effort=25 velocity=37
- added joint right_wrist_roll_joint: type revolute, parent right_elbow_link, child right_wrist_roll_rubber_hand, origin xyz=0.100 -0.00188791 -0.010 rpy=0 0 0, axis 1 0 0, limit lower=-1.972222054 upper=1.972222054 effort=25 velocity=37
- added joint waist_support_joint: type fixed, parent torso_link, child waist_support_link, origin xyz=0.0039635 0 -0.054 rpy=0 0 0
- added joint waist_yaw_fixed_joint: type fixed, parent torso_link, child waist_yaw_fixed_link, origin xyz=0.0039635 0 -0.054 rpy=0 0 0
- added joint waist_yaw_joint: type revolute, parent pelvis, child torso_link, origin xyz=-0.0039635 0 0.054 rpy=0 0 0, axis 0 0 1, limit lower=-2.618 upper=2.618 effort=88 velocity=32
- joint keyframe_head_joint: child Torso_Side_Right -> keyframe_head_link; origin xyz=-0.10 -0.10 -0.39 rpy=0 0 0 -> xyz=0 0 0.45 rpy=0 0 0; parent base -> torso_link
